File: at90s2323/Kicad/at90s2323.kicad_pcb (KiCad board)
At the start: 2 copper layers, 99.1 x 99.1 mm, 171 parts, among them J1 Barrel_Jack_Switch, J2 AVR-ISP-10, J3 Conn_01x04_Male, J4 Conn_01x04_Male, SW1 SW_Push, U1 74HC595, U2 74HC595, U3 TPIC6B595, U4 L7805, U5 AT90S2323, U6 MAX809M, Y1 10MHz

Commit message: Convert to Kicad 6
Connections:
- net ~RESET renamed ~{RESET}
Other:
- net class Default removed
- board text added: "~{RESET}"
- board text removed: "~RESET"

Commit message: Kicad 6 ERC fixes.
Connections:
- D130 pad 2: Net-(D130-Pad2) -> unconnected-(D130-Pad2)
- J2 pad 3: Net-(J2-Pad3) -> unconnected-(J2-Pad3)
- U2 pad 9: Net-(U2-Pad9) -> unconnected-(U2-Pad9)
