File: at90s2323/Kicad/at90s2323.kicad_sch (KiCad schematic)
At the start: 171 parts, among them J1 Barrel_Jack_Switch, J2 AVR-ISP-10, J3 Conn_01x04_Male, J4 Conn_01x04_Male, SW1 SW_Push, U1 74HC595, U2 74HC595, U3 TPIC6B595, U4 L7805, U5 AT90S2323, U6 MAX809M, Y1 10MHz

Commit message: Kicad 6 ERC fixes.
Parts:
- C3, C4: symbol Device:CP -> Device:C_Polarized
Changed lines of the file:
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@@
     (pin "3")
   )
-  (symbol (lib_id "Device:CP") (at 52.07 41.91 0) (unit 1)
+  (symbol (lib_id "Device:C_Polarized") (at 52.07 41.91 0) (unit 1)
     (in_bom yes) (on_board yes)
     (property "Reference" "C3" (id 0) (at 55.0672 40.7416 0)
@@
     (pin "2")
   )
-  (symbol (lib_id "Device:CP") (at 86.36 41.91 0) (unit 1)
+  (symbol (lib_id "Device:C_Polarized") (at 86.36 41.91 0) (unit 1)
     (in_bom yes) (on_board yes)
     (property "Reference" "C4" (id 0) (at 89.3572 40.7416 0)
