File: at90s8535/Kicad/Level translators.kicad_sch (KiCad schematic)
At the start: 8 parts, among them U3 74AHCT125D, U6 74AHCT125D, U8 74AHCT125D

Commit message: Correct part number for 5V to 3V level translation.
Parts:
- U11, U6: renamed from U8; value 74AHCT125D -> 74AHC125D
- U3: value 74AHCT125D -> 74AHC125D
- renumbered C13 to C18, C8 to C7, C13 to C8, U6 to U8
