File: at90s8535/Kicad/Programming debug.kicad_sch (KiCad schematic)
At the start: 10 parts, among them J1 AVR-ISP-6, J2 AVR-JTAG-10, SW1 SW_Push, U6 MAX809M

Commit message: Exclude solder jumper from BOM.
Parts:
- JP1: now left out of the parts list
Changed lines of the file:
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@@
   )
   (symbol (lib_id "Jumper:SolderJumper_2_Bridged") (at 52.07 110.49 0) (unit 1)
-    (in_bom yes) (on_board yes) (dnp no) (fields_autoplaced)
+    (in_bom no) (on_board yes) (dnp no) (fields_autoplaced)
     (property "Reference" "JP1" (at 52.07 107.95 0)
       (effects (font (size 1.27 1.27)))

Commit message: Change LED R from 1k to 10k.
Parts:
- R13: value 1k -> 10k
Changed lines of the file:
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@@
   (symbol (lib_id "Device:R") (at 185.42 66.04 0) (unit 1)
     (in_bom yes) (on_board yes) (dnp no) (fields_autoplaced)
-    (property "Reference" "R13" (at 182.88 65.405 0)
-      (effects (font (size 1.27 1.27)) (justify right))
+    (property "Reference" "R13" (at 187.96 65.405 0)
+      (effects (font (size 1.27 1.27)) (justify left))
     )
-    (property "Value" "1k" (at 182.88 67.945 0)
-      (effects (font (size 1.27 1.27)) (justify right))
+    (property "Value" "10k" (at 187.96 67.945 0)
+      (effects (font (size 1.27 1.27)) (justify left))
     )
     (property "Footprint" "Resistor_SMD:R_0805_2012Metric_Pad1.20x1.40mm_HandSolder" (at 183.642 66.04 90)

Commit message: Correct part number for 5V to 3V level translation.
Parts:
- renumbered D2 to D8, R13 to R16
Changed lines of the file:
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@@
     (instances
       (project "at90s8535"
-        (path "/b25be410-ef2b-47a5-b0e7-4e30ab693d4d"
+        (path "/b25be410-ef2b-47a5-b0e7-4e30ab693d4d/1e646dbe-cff2-478d-8c98-86d3163284b6"
           (reference "SW1") (unit 1)
         )
-        (path "/b25be410-ef2b-47a5-b0e7-4e30ab693d4d/1e646dbe-cff2-478d-8c98-86d3163284b6"
-          (reference "SW1") (unit 1)
-        )
       )
     )
@@
   (symbol (lib_id "Device:LED") (at 185.42 53.34 90) (unit 1)
     (in_bom yes) (on_board yes) (dnp no) (fields_autoplaced)
-    (property "Reference" "D2" (at 189.23 54.2925 90)
+    (property "Reference" "D8" (at 189.23 54.2925 90)
       (effects (font (size 1.27 1.27)) (justify right))
     )
@@
     (instances
       (project "at90s8535"
-        (path "/b25be410-ef2b-47a5-b0e7-4e30ab693d4d"
-          (reference "D2") (unit 1)
-        )
         (path "/b25be410-ef2b-47a5-b0e7-4e30ab693d4d/1e646dbe-cff2-478d-8c98-86d3163284b6"
           (reference "D8") (unit 1)
@@
     (instances
       (project "at90s8535"
-        (path "/b25be410-ef2b-47a5-b0e7-4e30ab693d4d"
+        (path "/b25be410-ef2b-47a5-b0e7-4e30ab693d4d/1e646dbe-cff2-478d-8c98-86d3163284b6"
           (reference "J2") (unit 1)
         )
-        (path "/b25be410-ef2b-47a5-b0e7-4e30ab693d4d/1e646dbe-cff2-478d-8c98-86d3163284b6"
-          (reference "J2") (unit 1)
-        )
       )
     )
@@
     (instances
       (project "at90s8535"
-        (path "/b25be410-ef2b-47a5-b0e7-4e30ab693d4d"
+        (path "/b25be410-ef2b-47a5-b0e7-4e30ab693d4d/1e646dbe-cff2-478d-8c98-86d3163284b6"
           (reference "#PWR06") (unit 1)
         )
-        (path "/b25be410-ef2b-47a5-b0e7-4e30ab693d4d/1e646dbe-cff2-478d-8c98-86d3163284b6"
-          (reference "#PWR06") (unit 1)
-        )
       )
     )
@@
     (instances
       (project "at90s8535"
-        (path "/b25be410-ef2b-47a5-b0e7-4e30ab693d4d"
-          (reference "C17") (unit 1)
-        )
         (path "/b25be410-ef2b-47a5-b0e7-4e30ab693d4d/1e646dbe-cff2-478d-8c98-86d3163284b6"
           (reference "C17") (unit 1)
@@
   (symbol (lib_id "power:GND") (at 90.17 78.74 0) (unit 1)
     (in_bom yes) (on_board yes) (dnp no) (fields_autoplaced)
-    (property "Reference" "#PWR05" (at 90.17 85.09 0)
+    (property "Reference" "#PWR07" (at 90.17 85.09 0)
       (effects (font (size 1.27 1.27)) hide)
     )
@@
     (instances
       (project "at90s8535"
-        (path "/b25be410-ef2b-47a5-b0e7-4e30ab693d4d"
-          (reference "#PWR05") (unit 1)
-        )
         (path "/b25be410-ef2b-47a5-b0e7-4e30ab693d4d/1e646dbe-cff2-478d-8c98-86d3163284b6"
           (reference "#PWR07") (unit 1)
@@
   (symbol (lib_id "Device:R") (at 185.42 66.04 0) (unit 1)
     (in_bom yes) (on_board yes) (dnp no) (fields_autoplaced)
-    (property "Reference" "R13" (at 187.96 65.405 0)
+    (property "Reference" "R16" (at 187.96 65.405 0)
       (effects (font (size 1.27 1.27)) (justify left))
     )
@@
     (instances
       (project "at90s8535"
-        (path "/b25be410-ef2b-47a5-b0e7-4e30ab693d4d"
-          (reference "R13") (unit 1)
-        )
         (path "/b25be410-ef2b-47a5-b0e7-4e30ab693d4d/1e646dbe-cff2-478d-8c98-86d3163284b6"
           (reference "R16") (unit 1)
@@
     (instances
       (project "at90s8535"
-        (path "/b25be410-ef2b-47a5-b0e7-4e30ab693d4d"
-          (reference "#PWR060") (unit 1)
-        )
         (path "/b25be410-ef2b-47a5-b0e7-4e30ab693d4d/1e646dbe-cff2-478d-8c98-86d3163284b6"
           (reference "#PWR060") (unit 1)
@@
     (instances
       (project "at90s8535"
-        (path "/b25be410-ef2b-47a5-b0e7-4e30ab693d4d"
-          (reference "J1") (unit 1)
-        )
         (path "/b25be410-ef2b-47a5-b0e7-4e30ab693d4d/1e646dbe-cff2-478d-8c98-86d3163284b6"
           (reference "J1") (unit 1)
@@
     (instances
       (project "at90s8535"
-        (path "/b25be410-ef2b-47a5-b0e7-4e30ab693d4d"
-          (reference "JP1") (unit 1)
-        )
         (path "/b25be410-ef2b-47a5-b0e7-4e30ab693d4d/1e646dbe-cff2-478d-8c98-86d3163284b6"
           (reference "JP1") (unit 1)
@@
   (symbol (lib_id "power:GND") (at 38.1 78.74 0) (unit 1)
     (in_bom yes) (on_board yes) (dnp no) (fields_autoplaced)
-    (property "Reference" "#PWR04" (at 38.1 85.09 0)
+    (property "Reference" "#PWR05" (at 38.1 85.09 0)
       (effects (font (size 1.27 1.27)) hide)
     )
@@
     (instances
       (project "at90s8535"
-        (path "/b25be410-ef2b-47a5-b0e7-4e30ab693d4d"
-          (reference "#PWR04") (unit 1)
-        )
         (path "/b25be410-ef2b-47a5-b0e7-4e30ab693d4d/1e646dbe-cff2-478d-8c98-86d3163284b6"
           (reference "#PWR05") (unit 1)
@@
   (symbol (lib_id "power:+5V") (at 38.1 38.1 0) (unit 1)
     (in_bom yes) (on_board yes) (dnp no) (fields_autoplaced)
-    (property "Reference" "#PWR07" (at 38.1 41.91 0)
+    (property "Reference" "#PWR04" (at 38.1 41.91 0)
       (effects (font (size 1.27 1.27)) hide)
     )
@@
     (instances
       (project "at90s8535"
-        (path "/b25be410-ef2b-47a5-b0e7-4e30ab693d4d"
-          (reference "#PWR07") (unit 1)
-        )
         (path "/b25be410-ef2b-47a5-b0e7-4e30ab693d4d/1e646dbe-cff2-478d-8c98-86d3163284b6"
           (reference "#PWR04") (unit 1)
@@
     (instances
       (project "at90s8535"
-        (path "/b25be410-ef2b-47a5-b0e7-4e30ab693d4d"
+        (path "/b25be410-ef2b-47a5-b0e7-4e30ab693d4d/1e646dbe-cff2-478d-8c98-86d3163284b6"
           (reference "#PWR010") (unit 1)
-        )
-        (path "/b25be410-ef2b-47a5-b0e7-4e30ab693d4d/1e646dbe-cff2-478d-8c98-86d3163284b6"
-          (reference "#PWR010") (unit 1)
