File: at90s8535/Kicad/at90s8535.kicad_pcb (KiCad board)
At the start: 2 copper layers, 99.1 x 99.1 mm, 46 parts, among them J1 AVR-ISP-6, J10 Pmod host SPI, J2 AVR-JTAG-10, J3 Barrel_Jack_Switch, J4 Pmod host UART, J5 Pmod host SPI, J6 Pmod host I2C, J7 Pmod host GPIO, J8 Pmod host GPIO, J9 Pmod host SPI, SW1 SW_Push, U1 AT90S8535-8PC, U11 74AHCT125D, U2 L7805, U3 74AHCT125D, U4 AMS1117-3.3, U5 MAX809M, U6 74AHCT125D, U8 74AHCT125D, Y1 8MHz

Commit message: Change LED R from 1k to 10k.
Parts:
- R16: value 1k -> 10k
Changed lines of the file:
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@@
         (effects (font (size 1 1) (thickness 0.15)) (justify mirror))
     )
-    (fp_text value "1k" (at 0 -1.65) (layer "B.Fab")
+    (fp_text value "10k" (at 0 -1.65) (layer "B.Fab")
         (effects (font (size 1 1) (thickness 0.15)) (justify mirror))
     )

Commit message: Correct part number for 5V to 3V level translation.
Parts:
- U11, U3, U6: value 74AHCT125D -> 74AHC125D
