File: at90s1200/Kicad/at90s1200.kicad_pcb (KiCad board)
At the start: 2 copper layers, 99.1 x 99.1 mm, 34 parts, among them J1 AVR-ISP-10, J2 Barrel_Jack_Switch, J3 Conn_01x10_Male, J4 Conn_01x10_Male, SW1 SW_Push, SW2 SW_Push, U1 AT90S1200, U2 L7805, Y1 8MHz

Commit message: Convert to Kicad 6
Connections:
- net ~RESET renamed ~{RESET}
Other:
- net class Default removed
- board text added: "~{RESET}"
- board text removed: "~RESET"

Commit message: Kicad 6 ERC fixes.
Connections:
- J1 pad 3: Net-(J1-Pad3) -> unconnected-(J1-Pad3)
Other:
- board text removed: "JLCJLCJLCJLC"

Commit message: Redraw schematic to contain actual schema instead of only labels. Kicad upgrade. No change to board.
Parts:
- U1: value AT90S1200 -> AT90S1200-12PC
Connections:
- net VCC renamed +5V
Other:
- board text added: "${TITLE}"
- board text added: "http://atoomnet.net/ ${ISSUE_DATE}"
- board text removed: "AT90S1200/AT90S2313 demo board"
- board text removed: "http://atoomnet.net/ 2020-12-11"
