File: at90s1200/Kicad/at90s1200.kicad_sch (KiCad schematic)
At the start: 34 parts, among them J1 AVR-ISP-10, J2 Barrel_Jack_Switch, J3 Conn_01x10_Male, J4 Conn_01x10_Male, SW1 SW_Push, SW2 SW_Push, U1 AT90S1200, U2 L7805, Y1 8MHz

Commit message: Kicad 6 ERC fixes.
Parts:
- C3, C4: symbol Device:CP -> Device:C_Polarized
- D3, D4: symbol Device:LED_BCRG -> Device:LED_BKRG
Changed lines of the file:
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@@
   (junction (at 86.36 31.75) (diameter 0) (color 0 0 0 0)
   )
+  (junction (at 31.75 48.26) (diameter 0) (color 0 0 0 0)
+  )
   (wire (pts (xy 236.22 78.74) (xy 236.22 76.2))
     (stroke (width 0) (type default) (color 0 0 0 0))
@@
     (stroke (width 0) (type default) (color 0 0 0 0))
   )
+  (wire (pts (xy 31.75 48.26) (xy 31.75 53.34))
+    (stroke (width 0) (type default) (color 0 0 0 0))
+  )
   (wire (pts (xy 29.21 31.75) (xy 36.83 31.75))
     (stroke (width 0) (type default) (color 0 0 0 0))
@@
     (stroke (width 0) (type default) (color 0 0 0 0))
   )
+  (wire (pts (xy 35.56 48.26) (xy 35.56 53.34))
+    (stroke (width 0) (type default) (color 0 0 0 0))
+  )
   (wire (pts (xy 177.8 100.33) (xy 177.8 114.3))
     (stroke (width 0) (type default) (color 0 0 0 0))
@@
     (stroke (width 0) (type default) (color 0 0 0 0))
   )
-  (wire (pts (xy 31.75 36.83) (xy 31.75 53.34))
+  (wire (pts (xy 31.75 36.83) (xy 31.75 48.26))
     (stroke (width 0) (type default) (color 0 0 0 0))
   )
@@
     (stroke (width 0) (type default) (color 0 0 0 0))
   )
+  (wire (pts (xy 31.75 48.26) (xy 35.56 48.26))
+    (stroke (width 0) (type default) (color 0 0 0 0))
+  )
   (wire (pts (xy 128.27 106.68) (xy 135.89 106.68))
     (stroke (width 0) (type default) (color 0 0 0 0))
@@
   )
   (wire (pts (xy 125.73 168.91) (xy 129.54 168.91))
+    (stroke (width 0) (type default) (color 0 0 0 0))
+  )
+  (wire (pts (xy 52.07 22.86) (xy 52.07 31.75))
     (stroke (width 0) (type default) (color 0 0 0 0))
   )
@@
     (pin "3")
   )
-  (symbol (lib_id "Device:CP") (at 52.07 41.91 0) (unit 1)
+  (symbol (lib_id "Device:C_Polarized") (at 52.07 41.91 0) (unit 1)
     (in_bom yes) (on_board yes)
     (property "Reference" "C3" (id 0) (at 55.0672 40.7416 0)
@@
     (pin "2")
   )
-  (symbol (lib_id "Device:CP") (at 86.36 41.91 0) (unit 1)
+  (symbol (lib_id "Device:C_Polarized") (at 86.36 41.91 0) (unit 1)
     (in_bom yes) (on_board yes)
     (property "Reference" "C4" (id 0) (at 89.3572 40.7416 0)
@@
     (pin "1")
   )
-  (symbol (lib_id "Device:LED_BCRG") (at 120.65 176.53 90) (unit 1)
+  (symbol (lib_id "Device:LED_BKRG") (at 120.65 176.53 90) (unit 1)
     (in_bom yes) (on_board yes)
     (property "Reference" "D3" (id 0) (at 129.032 175.3616 90)
@@
     (pin "2")
   )
-  (symbol (lib_id "Device:LED_BCRG") (at 151.13 176.53 90) (unit 1)
+  (symbol (lib_id "Device:LED_BKRG") (at 151.13 176.53 90) (unit 1)
     (in_bom yes) (on_board yes)
     (property "Reference" "D4" (id 0) (at 159.512 175.3616 90)
@@
     (pin "1")
   )
+  (symbol (lib_id "power:PWR_FLAG") (at 52.07 22.86 0) (unit 1)
+    (in_bom yes) (on_board yes) (fields_autoplaced)
+    (property "Reference" "#FLG0101" (id 0) (at 52.07 20.955 0)
+      (effects (font (size 1.27 1.27)) hide)
+    )
+    (property "Value" "PWR_FLAG" (id 1) (at 52.07 17.78 0))
+    (property "Footprint" "" (id 2) (at 52.07 22.86 0)
+      (effects (font (size 1.27 1.27)) hide)
+    )
+    (property "Datasheet" "~" (id 3) (at 52.07 22.86 0)
+      (effects (font (size 1.27 1.27)) hide)
+    )
+    (pin "1")
+  )
+  (symbol (lib_id "power:PWR_FLAG") (at 35.56 53.34 180) (unit 1)
+    (in_bom yes) (on_board yes) (fields_autoplaced)
+    (property "Reference" "#FLG0102" (id 0) (at 35.56 55.245 0)
+      (effects (font (size 1.27 1.27)) hide)
+    )
+    (property "Value" "PWR_FLAG" (id 1) (at 38.1 54.6099 0)
+      (effects (font (size 1.27 1.27)) (justify right))
+    )
+    (property "Footprint" "" (id 2) (at 35.56 53.34 0)
+      (effects (font (size 1.27 1.27)) hide)
+    )
+    (property "Datasheet" "~" (id 3) (at 35.56 53.34 0)
+      (effects (font (size 1.27 1.27)) hide)
+    )
+    (pin "1")
+  )
   (sheet_instances
     (path "/" (page "1"))
   )
   (symbol_instances
+    (path "/297a413b-8372-49d7-a3cc-b20b59ff6c53"
+      (reference "#FLG0101") (unit 1) (value "PWR_FLAG") (footprint "")
+    )
+    (path "/53cd6ec5-664c-4312-b5fc-dde0611e05a4"
+      (reference "#FLG0102") (unit 1) (value "PWR_FLAG") (footprint "")
+    )
     (path "/00000000-0000-0000-0000-00005fd458e2"
       (reference "#PWR01") (unit 1) (value "GND") (footprint "")

Commit message: Redraw schematic to contain actual schema instead of only labels. Kicad upgrade. No change to board.
Parts:
- J3, J4: symbol Connector:Conn_01x10_Male -> Connector:Conn_01x10_Pin
- U1: value AT90S1200 -> AT90S1200-12PC
Other:
- company: (none) -> https://github.com/atoomnetmarc/AVR-demo-board/
- title: (none) -> AT90S1200/AT90S2313 demo board
- moved on the sheet: C1, C2, C5, C6, C7, D3, D4, J1, J3, J4, R10, R2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
